Commit message: ROS restructuring
Former-commit-id: 4aaa4337afb9b2309b2bbc7a5dbfe87fc9f8b023

File: ROS/UR5/ur5_path_planning/ur5_custom_description/urdf/ur5_on_table.xacro (robot description, xacro)
@@ -4,9 +4,17 @@
   <xacro:include filename="$(find ur_description)/urdf/common.gazebo.xacro"/>
   <!-- ur5 -->
+  <xacro:include filename="$(find ur5_custom_description)/urdf/ur5_vel_transmission.xacro" />
   <xacro:include filename="$(find ur_description)/urdf/ur5.urdf.xacro"/>
   <xacro:ur5_robot prefix="" joint_limited="true"/>
+  <xacro:ur5_vel_transmission prefix="" />
   <material name="blue">
     <color rgba="0 0 .8 1"/>
   </material>
+  <link name="world" />
+  <joint name="world_joint"  type="fixed">
+    <origin xyz="2 0 1.5" rpy="0 0 0" />
+    <parent link="world"/>
+    <child link="base_link_box"/>
+  </joint>
   <link name="base_link_box">
     <visual>
